Commit message: Add beer fetching demo objective
* Add scene and wrist camera
* Update controllers and groups for full-body waypoint control,
  single-chain cartesian control, and base-only/arm-only control.
* Use joint_state_broadcaster for base link joints instead of odom
  republisher script
* update lift limits
* Add odom offset republisher node to enable resetting odom without
  restarting the platform process.
* Add dependencies so dev source build works
* Add waypoints for demo
* Add ML models for segmentation in demo

File: src/dual_arm_mobile_hw/description/dual_arm_mobile_hw.urdf (robot description, URDF)
Before this commit: robot r100-0599, 131 links, 130 joints
Joints:
- joint linear_x_joint: limit lower=-100.0 upper=100.0 effort=1000.0 velocity=0.175 -> lower=-100.0 upper=100.0 effort=1000.0 velocity=0.2
- joint linear_y_joint: limit lower=-100.0 upper=100.0 effort=1000.0 velocity=0.175 -> lower=-100.0 upper=100.0 effort=1000.0 velocity=0.2
- joint rotational_yaw_joint: limit effort=150.0 velocity=0.5235987755982988 -> effort=150.0 velocity=0.2
