Commit message: Teleop working except for pose jog

File: src/dual_arm_mobile_sim/description/dual_arm_mobile_sim.urdf.xacro (robot description, xacro)
@@ -105,4 +105,16 @@
   >
   </xacro:robotiq_2f85>
+  <!-- <link name="mobile_base_ee_link"/>
+  <joint name="mobile_base_ee_joint" type="fixed">
+    <origin rpy="0 0 0" xyz="0.0 0.0 0.5"/>
+    <parent link="chassis_link"/>
+    <child link="mobile_base_ee_link"/>
+  </joint>
+  <link name="mobile_base_ee_child_link"/>
+  <joint name="mobile_base_ee_child_joint" type="fixed">
+    <origin rpy="0 0 0" xyz="0.0 0.0 0.0"/>
+    <parent link="mobile_base_ee_link"/>
+    <child link="mobile_base_ee_child_link"/>
+  </joint> -->
   <ros2_control name="ur_mujoco_control" type="system">
     <hardware>

Commit message: Upgrade sim and hw configs from 8.7 to 8.9 (#11)
* Teleop working except for pose jog

* Add some mujoco frame debugging

* separates hatch and trainer, relocates trainer, removes hatch from the setup

* adds bottle to the scene

* Pose jog seems to work now with the updated SwitchControllers logic

* Update moveit_pro run command for simulation

* bottle sites added

* move bottle to table edge

* adds missing kinematics entry to JTC and configs, update bottle sites, updates test behavior

* gripper behaviors

* Add mujoco reset capabilities

* Start of hw config inheritance from sim config

* allow using mock hardware option for lift colums

* add display instructions to readme

* remove unused HW ros2_control.yaml

* fix typo in config.yaml, add fake lift hw, add arm hash codes, adds missing groups to srdf

* add correct moveit_pro run sim name

* move table in front of robot, adds look at table waypoint, relocate bottle, update mujoco keyframe

* successfull pick

* readme link fix

* Add more hw startup details

* pre-commit

* Remove commented out references to removed controllers

---------

Co-authored-by: sinaaghli <sina.aghli@gmail.com>
Co-authored-by: Breelyn Styler <breelyn.styler@picknik.ai>

File: src/dual_arm_mobile_sim/description/dual_arm_mobile_sim.urdf.xacro (robot description, xacro)
@@ -1,4 +1,4 @@
 <?xml version="1.0" ?>
-<robot name="r100-0599" xmlns:xacro="http://wiki.ros.org/xacro">
+<robot name="phoebe" xmlns:xacro="http://wiki.ros.org/xacro">
   <!-- Args that users may need to change. -->
   <xacro:arg name="mujoco_model" default=""/>
@@ -105,4 +105,16 @@
   >
   </xacro:robotiq_2f85>
+  <!-- <link name="mobile_base_ee_link"/>
+  <joint name="mobile_base_ee_joint" type="fixed">
+    <origin rpy="0 0 0" xyz="0.0 0.0 0.5"/>
+    <parent link="chassis_link"/>
+    <child link="mobile_base_ee_link"/>
+  </joint>
+  <link name="mobile_base_ee_child_link"/>
+  <joint name="mobile_base_ee_child_joint" type="fixed">
+    <origin rpy="0 0 0" xyz="0.0 0.0 0.0"/>
+    <parent link="mobile_base_ee_link"/>
+    <child link="mobile_base_ee_child_link"/>
+  </joint> -->
   <ros2_control name="ur_mujoco_control" type="system">
     <hardware>
@@ -110,4 +122,5 @@
       <param name="mujoco_model">$(arg mujoco_model)</param>
       <param name="mujoco_model_package">dual_arm_mobile_sim</param>
+      <param name="mujoco_viewer">true</param>
       <param name="render_publish_rate">60</param>
       <param name="tf_publish_rate">60</param>
