Commit message: Rename dual_arm_mobile_* to phoebe_*

File: src/phoebe_bridgeback_description/xacro/clearpath_r100.macro.xacro (robot description, xacro)
@@ -457,5 +457,5 @@
       <visual>
         <geometry>
-          <mesh filename="package://dual_arm_mobile_description/meshes/lift_rails.STL"/>
+          <mesh filename="package://phoebe_description/meshes/lift_rails.STL"/>
         </geometry>
         <material name="clearpath_dark_grey"/>
@@ -477,5 +477,5 @@
       <visual>
         <geometry>
-          <mesh filename="package://dual_arm_mobile_description/meshes/shelf.STL"/>
+          <mesh filename="package://phoebe_description/meshes/shelf.STL"/>
         </geometry>
         <material name="clearpath_dark_grey"/>
@@ -497,5 +497,5 @@
       <visual>
         <geometry>
-          <mesh filename="package://dual_arm_mobile_description/meshes/shelf.STL"/>
+          <mesh filename="package://phoebe_description/meshes/shelf.STL"/>
         </geometry>
         <material name="clearpath_dark_grey"/>
@@ -517,5 +517,5 @@
       <visual>
         <geometry>
-          <mesh filename="package://dual_arm_mobile_description/meshes/monitor_hinge_base.STL"/>
+          <mesh filename="package://phoebe_description/meshes/monitor_hinge_base.STL"/>
         </geometry>
         <material name="clearpath_dark_grey"/>
@@ -537,5 +537,5 @@
       <visual>
         <geometry>
-          <mesh filename="package://dual_arm_mobile_description/meshes/monitor_hinge_top.STL"/>
+          <mesh filename="package://phoebe_description/meshes/monitor_hinge_top.STL"/>
         </geometry>
         <material name="clearpath_dark_grey"/>
@@ -557,5 +557,5 @@
       <visual>
         <geometry>
-          <mesh filename="package://dual_arm_mobile_description/meshes/monitor.STL"/>
+          <mesh filename="package://phoebe_description/meshes/monitor.STL"/>
         </geometry>
         <material name="clearpath_dark_grey"/>
@@ -577,5 +577,5 @@
       <visual>
         <geometry>
-          <mesh filename="package://dual_arm_mobile_description/meshes/monitor.STL"/>
+          <mesh filename="package://phoebe_description/meshes/monitor.STL"/>
         </geometry>
         <material name="clearpath_dark_grey"/>
@@ -597,5 +597,5 @@
       <visual>
         <geometry>
-          <mesh filename="package://dual_arm_mobile_description/meshes/ur_control_box.STL"/>
+          <mesh filename="package://phoebe_description/meshes/ur_control_box.STL"/>
         </geometry>
         <material name="clearpath_aluminum"/>
@@ -617,5 +617,5 @@
       <visual>
         <geometry>
-          <mesh filename="package://dual_arm_mobile_description/meshes/ur_control_box.STL"/>
+          <mesh filename="package://phoebe_description/meshes/ur_control_box.STL"/>
         </geometry>
         <material name="clearpath_aluminum"/>
@@ -637,5 +637,5 @@
       <visual>
         <geometry>
-          <mesh filename="package://dual_arm_mobile_description/meshes/scu.STL"/>
+          <mesh filename="package://phoebe_description/meshes/scu.STL"/>
         </geometry>
         <material name="clearpath_aluminum"/>
@@ -657,5 +657,5 @@
       <visual>
         <geometry>
-          <mesh filename="package://dual_arm_mobile_description/meshes/scu.STL"/>
+          <mesh filename="package://phoebe_description/meshes/scu.STL"/>
         </geometry>
         <material name="clearpath_aluminum"/>
@@ -677,5 +677,5 @@
       <visual>
         <geometry>
-          <mesh filename="package://dual_arm_mobile_description/meshes/autec_receiver.STL"/>
+          <mesh filename="package://phoebe_description/meshes/autec_receiver.STL"/>
         </geometry>
         <material name="clearpath_yellow"/>
@@ -697,5 +697,5 @@
       <visual>
         <geometry>
-          <mesh filename="package://dual_arm_mobile_description/meshes/wifi_antenna.STL"/>
+          <mesh filename="package://phoebe_description/meshes/wifi_antenna.STL"/>
         </geometry>
         <material name="clearpath_dark_grey"/>
@@ -717,5 +717,5 @@
       <visual>
         <geometry>
-          <mesh filename="package://dual_arm_mobile_description/meshes/wifi_antenna.STL"/>
+          <mesh filename="package://phoebe_description/meshes/wifi_antenna.STL"/>
         </geometry>
         <material name="clearpath_dark_grey"/>
@@ -737,5 +737,5 @@
       <visual>
         <geometry>
-          <mesh filename="package://dual_arm_mobile_description/meshes/autec_antenna.STL"/>
+          <mesh filename="package://phoebe_description/meshes/autec_antenna.STL"/>
         </geometry>
         <material name="clearpath_dark_grey"/>
@@ -757,11 +757,11 @@
       <visual>
         <geometry>
-          <mesh filename="package://dual_arm_mobile_description/meshes/arm_mount.STL"/>
-        </geometry>
-        <material name="clearpath_dark_grey"/>
-      </visual>
-      <collision>
-        <geometry>
-          <mesh filename="package://dual_arm_mobile_description/meshes/arm_mount_collision.STL"/>
+          <mesh filename="package://phoebe_description/meshes/arm_mount.STL"/>
+        </geometry>
+        <material name="clearpath_dark_grey"/>
+      </visual>
+      <collision>
+        <geometry>
+          <mesh filename="package://phoebe_description/meshes/arm_mount_collision.STL"/>
         </geometry>
       </collision>
@@ -776,11 +776,11 @@
       <visual>
         <geometry>
-          <mesh filename="package://dual_arm_mobile_description/meshes/arm_mount.STL"/>
-        </geometry>
-        <material name="clearpath_dark_grey"/>
-      </visual>
-      <collision>
-        <geometry>
-          <mesh filename="package://dual_arm_mobile_description/meshes/arm_mount_collision.STL"/>
+          <mesh filename="package://phoebe_description/meshes/arm_mount.STL"/>
+        </geometry>
+        <material name="clearpath_dark_grey"/>
+      </visual>
+      <collision>
+        <geometry>
+          <mesh filename="package://phoebe_description/meshes/arm_mount_collision.STL"/>
         </geometry>
       </collision>

File: src/phoebe_hw/description/phoebe_hw.urdf.xacro (robot description, xacro)
@@ -2,5 +2,15 @@
 <robot name="phoebe" xmlns:xacro="http://wiki.ros.org/xacro">
   <!-- Args that users may need to change. -->
-  <xacro:arg name="mujoco_model" default=""/>
+  <xacro:arg name="left_lift_comm_port" default="/dev/ttyUSB1"/>
+  <xacro:arg name="right_lift_comm_port" default="/dev/ttyUSB2"/>
+  <xacro:arg name="use_fake_lift_hardware" default="true"/>
+  <xacro:arg name="left_arm_ip" default="192.168.131.4"/>
+  <xacro:arg name="left_tool_device_name" default="/dev/ttyUSB0"/>
+  <xacro:arg name="right_arm_ip" default="192.168.131.3"/>
+  <xacro:arg name="right_tool_device_name" default="/tmp/ttyUR"/>
+  <xacro:arg name="left_gripper_comm_port" default="/dev/ttyUSB0"/>
+  <xacro:arg name="right_gripper_comm_port" default="/tmp/ttyUR"/>
+  <xacro:arg name="left_arm_kinematics_hash" default="calib_10848939019749023817"/>
+  <xacro:arg name="right_arm_kinematics_hash" default="calib_5972249097379105770"/>
   <!-- Mobile base joints -->
   <link name="world"/>
@@ -35,10 +45,10 @@
     <hardware>
       <plugin>clearpath_controller_interface/ClearpathControllerInterface</plugin>
-      <param name="odom_topic">/platform_velocity_controller/odom</param>
-      <param name="cmd_vel_topic">/platform_velocity_controller/cmd_vel_unstamped</param>
-      <param name="max_linear_velocity">0.2</param>
-      <param name="max_angular_velocity">0.2</param>
+      <param name="odom_topic">/r100_0599/platform/odom/offset</param>
+      <param name="cmd_vel_topic">/r100_0599/platform/cmd_vel_unstamped</param>
+      <param name="max_linear_velocity">1.0</param>
+      <param name="max_angular_velocity">1.0</param>
       <param name="cmd_pub_rate">50</param>
-      <param name="active_on_startup">true</param>
+      <param name="active_on_startup">false</param>
     </hardware>
     <joint name="linear_x_joint"/>
@@ -47,17 +57,19 @@
   </ros2_control>
   <!-- Mobile base -->
-  <xacro:include filename="$(find dual_arm_mobile_description)/xacro/clearpath_r100.macro.xacro"/>
+  <xacro:include filename="$(find phoebe_description)/xacro/clearpath_r100.macro.xacro"/>
   <xacro:clearpath_r100
       parent_link="base_link"
-      generate_ros2_control_tag="false"
+      generate_ros2_control_tag="true"
   >
   </xacro:clearpath_r100>
   <!-- Lifts -->
-  <xacro:include filename="$(find dual_arm_mobile_description)/xacro/ewellix_tlt500.macro.xacro"/>
+  <xacro:include filename="$(find phoebe_description)/xacro/ewellix_tlt500.macro.xacro" />
   <!-- Left lift -->
   <xacro:ewellix_tlt500
       parent_link="default_mount"
       prefix="lift_left_"
-      generate_ros2_control_tag="false"
+      generate_ros2_control_tag="true"
+      lift_comm_port="$(arg left_lift_comm_port)"
+      use_fake_lift_hardware="$(arg use_fake_lift_hardware)"
   >
     <origin rpy="0.0 0.0 0.0" xyz="0.0 0.2 0.04"/>
@@ -67,16 +79,26 @@
       parent_link="default_mount"
       prefix="lift_right_"
-      generate_ros2_control_tag="false"
+      generate_ros2_control_tag="true"
+      lift_comm_port="$(arg right_lift_comm_port)"
+      use_fake_lift_hardware="$(arg use_fake_lift_hardware)"
   >
     <origin rpy="0.0 0.0 0.0" xyz="0.0 -0.2 0.04"/>
   </xacro:ewellix_tlt500>
   <!-- Arms -->
-  <xacro:include filename="$(find dual_arm_mobile_description)/xacro/ur5e.macro.xacro"/>
+  <xacro:include filename="$(find phoebe_description)/xacro/ur5e.macro.xacro" />
   <!-- Left arm -->
   <xacro:ur5e
-      parent_link="left_arm_mount_plate_2"
-      prefix="left_"
-      generate_ros2_control_tag="false"
-  >
+    parent_link="left_arm_mount_plate_2"
+    prefix="left_"
+    generate_ros2_control_tag="true"
+    robot_ip="$(arg left_arm_ip)"
+    reverse_port="50001"
+    script_sender_port="50002"
+    script_command_port="50004"
+    trajectory_port="50003"
+    tool_device_name="$(arg left_tool_device_name)"
+    tool_tcp_port="54320"
+    kinematics_hash="$(arg left_arm_kinematics_hash)"
+    >
     <origin rpy="0 0 -0.7853981633974483" xyz="0 0 0"/>
   </xacro:ur5e>
@@ -85,15 +107,24 @@
       parent_link="right_arm_mount_plate_2"
       prefix="right_"
-      generate_ros2_control_tag="false"
+      generate_ros2_control_tag="true"
+      robot_ip="$(arg right_arm_ip)"
+      reverse_port="50005"
+      script_sender_port="50006"
+      script_command_port="50008"
+      trajectory_port="50007"
+      tool_device_name="$(arg right_tool_device_name)"
+      tool_tcp_port="54321"
+      kinematics_hash="$(arg right_arm_kinematics_hash)"
   >
     <origin rpy="0 0 -2.356194490192345" xyz="0 0 0"/>
   </xacro:ur5e>
   <!-- Grippers -->
-  <xacro:include filename="$(find dual_arm_mobile_description)/xacro/robotiq_2f85.macro.xacro"/>
+  <xacro:include filename="$(find phoebe_description)/xacro/robotiq_2f85.macro.xacro"/>
   <!-- Left gripper -->
   <xacro:robotiq_2f85
       parent_link="left_realsense_camera_adapter_tool0"
       prefix="left_"
-      generate_ros2_control_tag="false"
+      generate_ros2_control_tag="true"
+      gripper_comm_port="$(arg left_gripper_comm_port)"
   >
   </xacro:robotiq_2f85>
@@ -102,33 +133,7 @@
       parent_link="right_realsense_camera_adapter_tool0"
       prefix="right_"
-      generate_ros2_control_tag="false"
+      generate_ros2_control_tag="true"
+      gripper_comm_port="$(arg right_gripper_comm_port)"
   >
   </xacro:robotiq_2f85>
-  <!-- <link name="mobile_base_ee_link"/>
-  <joint name="mobile_base_ee_joint" type="fixed">
-    <origin rpy="0 0 0" xyz="0.0 0.0 0.5"/>
-    <parent link="chassis_link"/>
-    <child link="mobile_base_ee_link"/>
-  </joint>
-  <link name="mobile_base_ee_child_link"/>
-  <joint name="mobile_base_ee_child_joint" type="fixed">
-    <origin rpy="0 0 0" xyz="0.0 0.0 0.0"/>
-    <parent link="mobile_base_ee_link"/>
-    <child link="mobile_base_ee_child_link"/>
-  </joint> -->
-  <ros2_control name="ur_mujoco_control" type="system">
-    <hardware>
-      <plugin>picknik_mujoco_ros/MujocoSystem</plugin>
-      <param name="mujoco_model">$(arg mujoco_model)</param>
-      <param name="mujoco_model_package">dual_arm_mobile_sim</param>
-      <param name="mujoco_viewer">true</param>
-      <param name="render_publish_rate">60</param>
-      <param name="tf_publish_rate">60</param>
-      <param name="lidar_publish_rate">10</param>
-      <param name="ignore_joint_validation">linear_x_joint linear_y_joint rotational_yaw_joint</param>
-      <param name="publish_odom">true</param>
-      <param name="odom_child_frame">ridgeback_base_link</param>
-      <param name="odom_zero_z">true</param>
-    </hardware>
-  </ros2_control>
 </robot>

File: src/phoebe_sim/description/phoebe_sim.urdf.xacro (robot description, xacro)
@@ -2,15 +2,5 @@
 <robot name="phoebe" xmlns:xacro="http://wiki.ros.org/xacro">
   <!-- Args that users may need to change. -->
-  <xacro:arg name="left_lift_comm_port" default="/dev/ttyUSB1"/>
-  <xacro:arg name="right_lift_comm_port" default="/dev/ttyUSB2"/>
-  <xacro:arg name="use_fake_lift_hardware" default="true"/>
-  <xacro:arg name="left_arm_ip" default="192.168.131.4"/>
-  <xacro:arg name="left_tool_device_name" default="/dev/ttyUSB0"/>
-  <xacro:arg name="right_arm_ip" default="192.168.131.3"/>
-  <xacro:arg name="right_tool_device_name" default="/tmp/ttyUR"/>
-  <xacro:arg name="left_gripper_comm_port" default="/dev/ttyUSB0"/>
-  <xacro:arg name="right_gripper_comm_port" default="/tmp/ttyUR"/>
-  <xacro:arg name="left_arm_kinematics_hash" default="calib_10848939019749023817"/>
-  <xacro:arg name="right_arm_kinematics_hash" default="calib_5972249097379105770"/>
+  <xacro:arg name="mujoco_model" default=""/>
   <!-- Mobile base joints -->
   <link name="world"/>
@@ -45,10 +35,10 @@
     <hardware>
       <plugin>clearpath_controller_interface/ClearpathControllerInterface</plugin>
-      <param name="odom_topic">/r100_0599/platform/odom/offset</param>
-      <param name="cmd_vel_topic">/r100_0599/platform/cmd_vel_unstamped</param>
-      <param name="max_linear_velocity">1.0</param>
-      <param name="max_angular_velocity">1.0</param>
+      <param name="odom_topic">/platform_velocity_controller/odom</param>
+      <param name="cmd_vel_topic">/platform_velocity_controller/cmd_vel_unstamped</param>
+      <param name="max_linear_velocity">0.2</param>
+      <param name="max_angular_velocity">0.2</param>
       <param name="cmd_pub_rate">50</param>
-      <param name="active_on_startup">false</param>
+      <param name="active_on_startup">true</param>
     </hardware>
     <joint name="linear_x_joint"/>
@@ -57,19 +47,17 @@
   </ros2_control>
   <!-- Mobile base -->
-  <xacro:include filename="$(find dual_arm_mobile_description)/xacro/clearpath_r100.macro.xacro"/>
+  <xacro:include filename="$(find phoebe_description)/xacro/clearpath_r100.macro.xacro"/>
   <xacro:clearpath_r100
       parent_link="base_link"
-      generate_ros2_control_tag="true"
+      generate_ros2_control_tag="false"
   >
   </xacro:clearpath_r100>
   <!-- Lifts -->
-  <xacro:include filename="$(find dual_arm_mobile_description)/xacro/ewellix_tlt500.macro.xacro" />
+  <xacro:include filename="$(find phoebe_description)/xacro/ewellix_tlt500.macro.xacro"/>
   <!-- Left lift -->
   <xacro:ewellix_tlt500
       parent_link="default_mount"
       prefix="lift_left_"
-      generate_ros2_control_tag="true"
-      lift_comm_port="$(arg left_lift_comm_port)"
-      use_fake_lift_hardware="$(arg use_fake_lift_hardware)"
+      generate_ros2_control_tag="false"
   >
     <origin rpy="0.0 0.0 0.0" xyz="0.0 0.2 0.04"/>
@@ -79,26 +67,16 @@
       parent_link="default_mount"
       prefix="lift_right_"
-      generate_ros2_control_tag="true"
-      lift_comm_port="$(arg right_lift_comm_port)"
-      use_fake_lift_hardware="$(arg use_fake_lift_hardware)"
+      generate_ros2_control_tag="false"
   >
     <origin rpy="0.0 0.0 0.0" xyz="0.0 -0.2 0.04"/>
   </xacro:ewellix_tlt500>
   <!-- Arms -->
-  <xacro:include filename="$(find dual_arm_mobile_description)/xacro/ur5e.macro.xacro" />
+  <xacro:include filename="$(find phoebe_description)/xacro/ur5e.macro.xacro"/>
   <!-- Left arm -->
   <xacro:ur5e
-    parent_link="left_arm_mount_plate_2"
-    prefix="left_"
-    generate_ros2_control_tag="true"
-    robot_ip="$(arg left_arm_ip)"
-    reverse_port="50001"
-    script_sender_port="50002"
-    script_command_port="50004"
-    trajectory_port="50003"
-    tool_device_name="$(arg left_tool_device_name)"
-    tool_tcp_port="54320"
-    kinematics_hash="$(arg left_arm_kinematics_hash)"
-    >
+      parent_link="left_arm_mount_plate_2"
+      prefix="left_"
+      generate_ros2_control_tag="false"
+  >
     <origin rpy="0 0 -0.7853981633974483" xyz="0 0 0"/>
   </xacro:ur5e>
@@ -107,24 +85,15 @@
       parent_link="right_arm_mount_plate_2"
       prefix="right_"
-      generate_ros2_control_tag="true"
-      robot_ip="$(arg right_arm_ip)"
-      reverse_port="50005"
-      script_sender_port="50006"
-      script_command_port="50008"
-      trajectory_port="50007"
-      tool_device_name="$(arg right_tool_device_name)"
-      tool_tcp_port="54321"
-      kinematics_hash="$(arg right_arm_kinematics_hash)"
+      generate_ros2_control_tag="false"
   >
     <origin rpy="0 0 -2.356194490192345" xyz="0 0 0"/>
   </xacro:ur5e>
   <!-- Grippers -->
-  <xacro:include filename="$(find dual_arm_mobile_description)/xacro/robotiq_2f85.macro.xacro"/>
+  <xacro:include filename="$(find phoebe_description)/xacro/robotiq_2f85.macro.xacro"/>
   <!-- Left gripper -->
   <xacro:robotiq_2f85
       parent_link="left_realsense_camera_adapter_tool0"
       prefix="left_"
-      generate_ros2_control_tag="true"
-      gripper_comm_port="$(arg left_gripper_comm_port)"
+      generate_ros2_control_tag="false"
   >
   </xacro:robotiq_2f85>
@@ -133,7 +102,33 @@
       parent_link="right_realsense_camera_adapter_tool0"
       prefix="right_"
-      generate_ros2_control_tag="true"
-      gripper_comm_port="$(arg right_gripper_comm_port)"
+      generate_ros2_control_tag="false"
   >
   </xacro:robotiq_2f85>
+  <!-- <link name="mobile_base_ee_link"/>
+  <joint name="mobile_base_ee_joint" type="fixed">
+    <origin rpy="0 0 0" xyz="0.0 0.0 0.5"/>
+    <parent link="chassis_link"/>
+    <child link="mobile_base_ee_link"/>
+  </joint>
+  <link name="mobile_base_ee_child_link"/>
+  <joint name="mobile_base_ee_child_joint" type="fixed">
+    <origin rpy="0 0 0" xyz="0.0 0.0 0.0"/>
+    <parent link="mobile_base_ee_link"/>
+    <child link="mobile_base_ee_child_link"/>
+  </joint> -->
+  <ros2_control name="ur_mujoco_control" type="system">
+    <hardware>
+      <plugin>picknik_mujoco_ros/MujocoSystem</plugin>
+      <param name="mujoco_model">$(arg mujoco_model)</param>
+      <param name="mujoco_model_package">phoebe_sim</param>
+      <param name="mujoco_viewer">true</param>
+      <param name="render_publish_rate">60</param>
+      <param name="tf_publish_rate">60</param>
+      <param name="lidar_publish_rate">10</param>
+      <param name="ignore_joint_validation">linear_x_joint linear_y_joint rotational_yaw_joint</param>
+      <param name="publish_odom">true</param>
+      <param name="odom_child_frame">ridgeback_base_link</param>
+      <param name="odom_zero_z">true</param>
+    </hardware>
+  </ros2_control>
 </robot>
